Commit message: frame fix

File: tortoisebot/tortoisebot_description/models/urdf/tortoisebot_simple.xacro (robot description, xacro)
@@ -118,4 +118,10 @@
     </collision>
   </link>
+  <link name="camera_optical_link"/>
+  <joint name="camera_optical_joint" type="fixed">
+    <parent link="camera_link"/>
+    <child link="camera_optical_link"/>
+    <origin xyz="0 0 0" rpy="-1.57 0 -1.57"/>
+  </joint>
   <link name="camera_holder">
     <inertial>
@@ -183,11 +189,4 @@
     <child link="camera_link" />
   </joint>
-  <!-- <link name="camera_not_optical_link" /> -->
-  <!-- <joint name="camera_optical_joint" type="fixed">
-    <parent link="camera_link"/>
-    <child link="camera_link_optical"/>
-    <origin xyz="0 0 0" rpy="-1.5708 0 -1.5708"/>
-  </joint> -->
-  <!-- <link name="camera_link" /> -->
   <joint name="camera_tilt_joint" type="fixed">
     <origin xyz="0.03125 0.0 0.131063" rpy="0 0 0" />
